Commit message: add oscillators and phase-based rewards, some tuning

File: resources/robots/mit_humanoid/urdf/humanoid_F_sf_learnt.urdf (robot description, URDF)
Before this commit: robot humanoid, 21 links, 20 joints
Links:
- link left_foot: mass  0.279583 -> 0.434332672008075; geometry collision cylinder length=0.15 radius=0.02; visual mesh filename=meshes_v3/left_foot.stl scale=0.001 0.001 0.001
- link left_hip_abad: mass 1.199631 -> 1.10845642066563
- link left_hip_yaw: mass  0.842752 -> 1.03610198878872
- link left_lower_leg: mass 0.346291 -> 0.238357586915263; geometry collision cylinder length=0.13 radius=0.05; visual mesh filename=meshes_v3/left_leg_lower.stl scale=0.001 0.001 0.001
- link left_upper_leg: mass 2.634789 -> 2.9466623694791; geometry collision cylinder length=0.16 radius=0.035; visual mesh filename=meshes_v3/left_leg_upper.stl scale=0.001 0.001 0.001
- link right_foot: mass  0.279583 -> 0.48135110558567; geometry collision cylinder length=0.15 radius=0.02; visual mesh filename=meshes_v3/left_foot.stl scale=0.001 -0.001 0.001
- link right_hip_abad: mass 1.199631 -> 2.22134334871633
- link right_hip_yaw: mass  0.842752 -> 0.944770728939119
- link right_lower_leg: mass 0.346291 -> 0.224587667752391; geometry collision cylinder length=0.13 radius=0.05; visual mesh filename=meshes_v3/left_leg_lower.stl scale=0.001 -0.001 0.001
- link right_upper_leg: mass 2.634789 -> 3.20991362323237; geometry collision cylinder length=0.16 radius=0.035; visual mesh filename=meshes_v3/left_leg_upper.stl scale=0.001 -0.001 0.001
Joints:
- joint 01_right_hip_yaw: origin xyz=0 -0.082 0 rpy=0 -0.174533 0 -> xyz=-0.00565 -0.082 -0.05735 rpy=0 -0.174533 0
- joint 03_right_hip_pitch: origin xyz=0.08837 0.00284 -0.01385 rpy=0 -0.261799 0 -> xyz=0.07133 0.002 0.0 rpy=0 -0.261799 0
- joint 04_right_knee: origin xyz=-0.01306 0.0 -0.24916 rpy=0 0 0 -> xyz=0.0 0.0 -0.2666 rpy=0 0 0
- joint 05_right_ankle: limit lower=-1.5 upper=1.5 effort=68 velocity=24 -> lower=-0.97 upper=0.97 effort=68 velocity=24
- joint 06_left_hip_yaw: origin xyz=0 0.082 0 rpy=0 -0.174533 0 -> xyz=-0.00565 0.082 -0.05735 rpy=0 -0.174533 0
- joint 08_left_hip_pitch: origin xyz=0.08837 -0.00284 -0.01385 rpy=0 -0.261799 0 -> xyz=0.07133 -0.002 0.0 rpy=0 -0.261799 0
- joint 09_left_knee: origin xyz=-0.01306 0.0 -0.24916 rpy=0 0 0 -> xyz=0.0 0.0 -0.2666 rpy=0 0 0
- joint 10_left_ankle: limit lower=-1.5 upper=1.5 effort=68 velocity=24 -> lower=-0.97 upper=0.97 effort=68 velocity=24
- joint 11_right_shoulder_pitch: origin xyz=0.01911 -0.17608 0.30392 rpy=0 0 0 -> xyz=0.01346 -0.17608 0.24657 rpy=0 0 0
- joint 15_left_shoulder_pitch: origin xyz=0.01911 0.17608 0.30392 rpy=0 0 0 -> xyz=0.01346 0.17608 0.24657 rpy=0 0 0

Commit message: enable arms in learnt urdf diff --git a/gym/envs/mit_humanoid/mit_humanoid_config.py b/gym/envs/mit_humanoid/mit_humanoid_config.py index 54813f7..368f2c3 100644 --- a/gym/envs/mit_humanoid/mit_humanoid_config.py +++ b/gym/envs/mit_humanoid/mit_humanoid_config.py @@ -142,7 +142,7 @@ class MITHumanoidCfg(LeggedRobotCfg):      class asset(LeggedRobotCfg.asset):          file = (              "{LEGGED_GYM_ROOT_DIR}/resources/robots/" -            + "mit_humanoid/urdf/humanoid_R_sf.urdf" +            + "mit_humanoid/urdf/humanoid_F_sf_learnt.urdf"          )          # foot_collisionbox_names = ["foot"]          foot_name = "foot" @@ -289,12 +289,12 @@ class MITHumanoidRunnerCfg(LeggedRobotRunnerCfg):          use_clipped_value_loss = True          clip_param = 0.2          entropy_coef = 0.01 -        num_learning_epochs = 5 +        num_learning_epochs = 4          # * mini batch size = num_envs*nsteps / nminibatches          num_mini_batches = 4 -        learning_rate = 5.0e-5 +        learning_rate = 1.0e-6          schedule = "adaptive"  # could be adaptive, fixed -        gamma = 0.999 +        gamma = 0.99          lam = 0.95          desired_kl = 0.01          max_grad_norm = 1.0 diff --git a/resources/robots/mit_humanoid/urdf/humanoid_F_sf_learnt.urdf b/resources/robots/mit_humanoid/urdf/humanoid_F_sf_learnt.urdf index 5e76f34..98a0773 100644 --- a/resources/robots/mit_humanoid/urdf/humanoid_F_sf_learnt.urdf +++ b/resources/robots/mit_humanoid/urdf/humanoid_F_sf_learnt.urdf @@ -570,7 +570,7 @@ Simple Foot: foot approximated as single box-contact -->    </link>    <joint      name="15_left_shoulder_pitch" -    type="fixed"> +    type="revolute">      <origin        xyz="0.01346 0.17608 0.24657"        rpy="0 0 0" /> @@ -615,7 +615,7 @@ Simple Foot: foot approximated as single box-contact -->    </link>    <joint      name="16_left_shoulder_abad" -    type="fixed"> +    type="revolute">      <origin        xyz="0 .05760 0"        rpy="0.0 0 0" /> @@ -668,7 +668,7 @@ Simple Foot: foot approximated as single box-contact -->    </link>    <joint      name="17_left_shoulder_yaw" -    type="fixed"> +    type="revolute">      <origin        xyz="0 0 -.10250"        rpy="0.0 0 0" /> @@ -719,7 +719,7 @@ Simple Foot: foot approximated as single box-contact -->    </link>    <joint      name="18_left_elbow" -    type="fixed"> +    type="revolute">      <origin        xyz="0 0 -.15750"        rpy="0 0 0.0" /> @@ -798,7 +798,7 @@ Simple Foot: foot approximated as single box-contact -->    </link>    <joint      name="11_right_shoulder_pitch" -    type="fixed"> +    type="revolute">      <origin        xyz="0.01346 -0.17608 0.24657"        rpy="0 0 0" /> @@ -843,7 +843,7 @@ Simple Foot: foot approximated as single box-contact -->    </link>    <joint      name="12_right_shoulder_abad" -    type="fixed"> +    type="revolute">      <origin        xyz="0 -.05760 0"        rpy="0.0 0 0" /> @@ -896,7 +896,7 @@ Simple Foot: foot approximated as single box-contact -->    </link>    <joint      name="13_right_shoulder_yaw" -    type="fixed"> +    type="revolute">      <origin        xyz="0 0 -.10250"        rpy="0.0 0 0" /> @@ -947,7 +947,7 @@ Simple Foot: foot approximated as single box-contact -->    </link>    <joint      name="14_right_elbow" -    type="fixed"> +    type="revolute">      <origin        xyz="0 0 -.15750"        rpy="0 0 0.0" />

File: resources/robots/mit_humanoid/urdf/humanoid_F_sf_learnt.urdf (robot description, URDF)
Before this commit: robot humanoid, 21 links, 20 joints
Joints:
- joint 11_right_shoulder_pitch: type fixed -> revolute
- joint 12_right_shoulder_abad: type fixed -> revolute
- joint 13_right_shoulder_yaw: type fixed -> revolute
- joint 14_right_elbow: type fixed -> revolute
- joint 15_left_shoulder_pitch: type fixed -> revolute
- joint 16_left_shoulder_abad: type fixed -> revolute
- joint 17_left_shoulder_yaw: type fixed -> revolute
- joint 18_left_elbow: type fixed -> revolute
