Commit message: rename links and joints

File: resources/robots/mini_horse/urdf/mini_horse_simple.urdf (robot description, URDF)
Before this commit: robot mini_horse, 22 links, 21 joints
Links:
- removed link FL_hip
- removed link FL_shank
- removed link FL_thigh
- removed link FR_hip
- removed link FR_shank
- removed link FR_thigh
- removed link RL_hip
- removed link RL_shank
- removed link RL_thigh
- removed link RR_hip
- removed link RR_shank
- removed link RR_thigh
- added link FL_cannon, mass 3.0; collision box size=0.08 0.08 0.25; visual cylinder length=0.3 radius=0.04
- added link FL_forearm, mass 2.0; collision box size=0.15 0.15 0.4; visual cylinder length=0.46 radius=0.075
- added link FL_pastern, mass 2.5; collision box size=0.06 0.06 0.1; visual cylinder length=0.13 radius=0.03
- added link FR_cannon, mass 3.0; collision box size=0.08 0.08 0.25; visual cylinder length=0.3 radius=0.04
- added link FR_forearm, mass 2.0; collision box size=0.15 0.15 0.4; visual cylinder length=0.46 radius=0.075
- added link FR_pastern, mass 2.5; collision box size=0.06 0.06 0.1; visual cylinder length=0.13 radius=0.03
- added link RL_cannon, mass 3.0; collision box size=0.1 0.1 0.3; visual cylinder length=0.36 radius=0.05
- added link RL_forearm, mass 2.0; collision box size=0.175 0.175 0.4; visual cylinder length=0.46 radius=0.09
- added link RL_pastern, mass 2.5; collision box size=0.06 0.06 0.12; visual cylinder length=0.15 radius=0.03
- added link RR_cannon, mass 3.0; collision box size=0.1 0.1 0.3; visual cylinder length=0.36 radius=0.05
- added link RR_forearm, mass 2.0; collision box size=0.175 0.175 0.4; visual cylinder length=0.46 radius=0.09
- added link RR_pastern, mass 2.5; collision box size=0.06 0.06 0.12; visual cylinder length=0.15 radius=0.03
Joints:
- removed joint 2_fl_haa
- removed joint 2_fr_haa
- removed joint 2_rf_haa
- removed joint 2_rr_haa
- removed joint FL_fetlock_joint
- removed joint FL_hip_joint
- removed joint FL_hoof_joint
- removed joint FL_knee_joint
- removed joint FR_fetlock_joint
- removed joint FR_hip_joint
- removed joint FR_hoof_joint
- removed joint FR_knee_joint
- removed joint RL_fetlock_joint
- removed joint RL_hip_joint
- removed joint RL_hoof_joint
- removed joint RL_knee_joint
- removed joint RR_fetlock_joint
- removed joint RR_hip_joint
- removed joint RR_hoof_joint
- removed joint RR_knee_joint
- added joint FL_cfe: type revolute, parent FL_forearm, child FL_cannon, origin xyz=-0.08 0 -0.48, axis 0 1 0, limit lower=0 upper=3.0 effort=40 velocity=2.0
- added joint FL_ffe: type revolute, parent FL_shoulder, child FL_forearm, origin xyz=0 0 0.025 rpy=0 0 0, axis 0 1 0, limit lower=-1.7 upper=0.5 effort=50 velocity=2.0
- added joint FL_haa: type revolute, parent base_fh, child FL_shoulder, origin xyz=0.35 0.225 -0.23 rpy=0 0 0, axis 1 0 0, limit lower=-0.2 upper=0.2 effort=18 velocity=41
- added joint FL_hfe: type revolute, parent FL_pastern, child FL_hoof, origin xyz=0 0 -0.1, axis 0 1 0, limit lower=-0.3 upper=1.2 effort=20 velocity=2.0
- added joint FL_pfe: type revolute, parent FL_cannon, child FL_pastern, origin xyz=0.04 0 -0.32, axis 0 1 0, limit lower=-1.2 upper=0.5 effort=30 velocity=2.0
- added joint FR_cfe: type revolute, parent FR_forearm, child FR_cannon, origin xyz=-0.08 0 -0.48, axis 0 1 0, limit lower=0 upper=3.0 effort=40 velocity=2.0
- added joint FR_ffe: type revolute, parent FR_shoulder, child FR_forearm, origin xyz=0 -0.2 0.025 rpy=0 0 0, axis 0 1 0, limit lower=-1.7 upper=0.5 effort=50 velocity=2.0
- added joint FR_haa: type revolute, parent base_fh, child FR_shoulder, origin xyz=0.35 -0.225 -0.23 rpy=0 0 0, axis 1 0 0, limit lower=-0.2 upper=0.2 effort=18 velocity=41
- added joint FR_hfe: type revolute, parent FR_pastern, child FR_hoof, origin xyz=0 0 -0.1, axis 0 1 0, limit lower=-0.3 upper=1.2 effort=20 velocity=2.0
- added joint FR_pfe: type revolute, parent FR_cannon, child FR_pastern, origin xyz=0.04 0 -0.32, axis 0 1 0, limit lower=-1.2 upper=0.5 effort=30 velocity=2.0
- added joint RL_cfe: type revolute, parent RL_forearm, child RL_cannon, origin xyz=0.09 0 -0.4, axis 0 1 0, limit lower=-3.0 upper=0.0 effort=40 velocity=2.0
- added joint RL_ffe: type revolute, parent RL_shoulder, child RL_forearm, origin xyz=0 0.12 -0.05 rpy=0 0 0, axis 0 1 0, limit lower=-0.5 upper=1.5 effort=50 velocity=2.0
- added joint RL_haa: type revolute, parent base_bh, child RL_shoulder, origin xyz=-0.3 0.225 -0.43 rpy=0 0 0, axis 1 0 0, limit lower=-0.2 upper=0.2 effort=18 velocity=41
- added joint RL_hfe: type revolute, parent RL_pastern, child RL_hoof, origin xyz=0 0 -0.16, axis 0 1 0, limit lower=-0.3 upper=1.5 effort=20 velocity=2.0
- added joint RL_pfe: type revolute, parent RL_cannon, child RL_pastern, origin xyz=-0.04 0 -0.35, axis 0 1 0, limit lower=-1.0 upper=0.0 effort=30 velocity=2.0
- added joint RR_cfe: type revolute, parent RR_forearm, child RR_cannon, origin xyz=0.09 0 -0.4, axis 0 1 0, limit lower=-3.0 upper=0.0 effort=40 velocity=2.0
- added joint RR_ffe: type revolute, parent RR_shoulder, child RR_forearm, origin xyz=0 -0.12 -0.05 rpy=0 0 0, axis 0 1 0, limit lower=-0.5 upper=1.5 effort=50 velocity=2.0
- added joint RR_haa: type revolute, parent base_bh, child RR_shoulder, origin xyz=-0.3 -0.225 -0.43 rpy=0 0 0, axis 1 0 0, limit lower=-0.2 upper=0.2 effort=18 velocity=41
- added joint RR_hfe: type revolute, parent RR_pastern, child RR_hoof, origin xyz=0 0 -0.16, axis 0 1 0, limit lower=-0.3 upper=1.5 effort=20 velocity=2.0
- added joint RR_pfe: type revolute, parent RR_cannon, child RR_pastern, origin xyz=-0.04 0 -0.35, axis 0 1 0, limit lower=-1.0 upper=0.0 effort=30 velocity=2.0

Commit message: training works

File: resources/robots/mini_horse/urdf/mini_horse_simple.urdf (robot description, URDF)
Before this commit: robot mini_horse, 22 links, 21 joints
Links:
- link base_bh: mass 145.0 -> 20.0
- link base_fh: mass 345.0 -> 20.0

Commit message: train horse to stand still

File: resources/robots/mini_horse/urdf/mini_horse_simple.urdf (robot description, URDF)
Before this commit: robot mini_horse, 22 links, 21 joints
Links:
- removed link FL_cannon
- removed link FL_forearm
- removed link FL_hoof
- removed link FL_pastern
- removed link FL_shoulder
- removed link FR_cannon
- removed link FR_forearm
- removed link FR_hoof
- removed link FR_pastern
- removed link FR_shoulder
- removed link RL_cannon
- removed link RL_forearm
- removed link RL_hoof
- removed link RL_pastern
- removed link RL_shoulder
- added link LF_cannon, mass 1.0; collision box size=0.08 0.08 0.25; visual cylinder length=0.3 radius=0.04
- added link LF_forearm, mass 1.0; collision box size=0.15 0.15 0.4; visual cylinder length=0.46 radius=0.075
- added link LF_hoof, mass 0.2; collision box size=0.1 0.1 0.07; visual cylinder length=0.08 radius=0.05
- added link LF_pastern, mass 0.5; collision box size=0.06 0.06 0.1; visual cylinder length=0.13 radius=0.03
- added link LF_shoulder, mass 2.0; visual cylinder length=0.05 radius=0.075
- added link LR_cannon, mass 1.0; collision box size=0.1 0.1 0.3; visual cylinder length=0.36 radius=0.05
- added link LR_forearm, mass 1.0; collision box size=0.175 0.175 0.4; visual cylinder length=0.46 radius=0.09
- added link LR_hoof, mass 0.2; collision box size=0.1 0.1 0.09; visual cylinder length=0.1 radius=0.05
- added link LR_pastern, mass 0.5; collision box size=0.06 0.06 0.12; visual cylinder length=0.15 radius=0.03
- added link LR_shoulder, mass 2.0; visual cylinder length=0.05 radius=0.075
- added link RF_cannon, mass 1.0; collision box size=0.08 0.08 0.25; visual cylinder length=0.3 radius=0.04
- added link RF_forearm, mass 1.0; collision box size=0.15 0.15 0.4; visual cylinder length=0.46 radius=0.075
- added link RF_hoof, mass 0.2; collision box size=0.1 0.1 0.07; visual cylinder length=0.08 radius=0.05
- added link RF_pastern, mass 0.5; collision box size=0.06 0.06 0.1; visual cylinder length=0.13 radius=0.03
- added link RF_shoulder, mass 2.0; visual cylinder length=0.05 radius=0.075
- link RR_cannon: mass 3.0 -> 1.0
- link RR_forearm: mass 2.0 -> 1.0
- link RR_hoof: mass 1.0 -> 0.2
- link RR_pastern: mass 2.5 -> 0.5
- link base_bh: mass 20.0 -> 4.0
- link base_fh: mass 20.0 -> 8.0
Joints:
- removed joint FL_cfe
- removed joint FL_ffe
- removed joint FL_haa
- removed joint FL_hfe
- removed joint FL_pfe
- removed joint FR_cfe
- removed joint FR_ffe
- removed joint FR_haa
- removed joint FR_hfe
- removed joint FR_pfe
- removed joint RL_cfe
- removed joint RL_ffe
- removed joint RL_haa
- removed joint RL_hfe
- removed joint RL_pfe
- added joint LF_cfe: type revolute, parent LF_forearm, child LF_cannon, origin xyz=-0.08 0 -0.48, axis 0 1 0, limit lower=0 upper=3.0 effort=40 velocity=2.0
- added joint LF_ffe: type revolute, parent LF_shoulder, child LF_forearm, origin xyz=0 0 0.025 rpy=0 0 0, axis 0 1 0, limit lower=-1.7 upper=0.5 effort=50 velocity=2.0
- added joint LF_haa: type revolute, parent base_fh, child LF_shoulder, origin xyz=0.35 0.225 -0.23 rpy=0 0 0, axis 1 0 0, limit lower=-0.2 upper=0.2 effort=18 velocity=41
- added joint LF_hfe: type revolute, parent LF_pastern, child LF_hoof, origin xyz=0 0 -0.1, axis 0 1 0, limit lower=-0.3 upper=1.2 effort=20 velocity=2.0
- added joint LF_pfe: type revolute, parent LF_cannon, child LF_pastern, origin xyz=0.04 0 -0.32, axis 0 1 0, limit lower=-1.2 upper=0.5 effort=30 velocity=2.0
- added joint LR_cfe: type revolute, parent LR_forearm, child LR_cannon, origin xyz=0.09 0 -0.4, axis 0 1 0, limit lower=-3.0 upper=0.0 effort=40 velocity=2.0
- added joint LR_ffe: type revolute, parent LR_shoulder, child LR_forearm, origin xyz=0 0.12 -0.05 rpy=0 0 0, axis 0 1 0, limit lower=-0.5 upper=1.5 effort=50 velocity=2.0
- added joint LR_haa: type revolute, parent base_bh, child LR_shoulder, origin xyz=-0.3 0.225 -0.43 rpy=0 0 0, axis 1 0 0, limit lower=-0.2 upper=0.2 effort=18 velocity=41
- added joint LR_hfe: type revolute, parent LR_pastern, child LR_hoof, origin xyz=0 0 -0.16, axis 0 1 0, limit lower=-0.3 upper=1.5 effort=20 velocity=2.0
- added joint LR_pfe: type revolute, parent LR_cannon, child LR_pastern, origin xyz=-0.04 0 -0.35, axis 0 1 0, limit lower=-1.0 upper=0.0 effort=30 velocity=2.0
- added joint RF_cfe: type revolute, parent RF_forearm, child RF_cannon, origin xyz=-0.08 0 -0.48, axis 0 1 0, limit lower=0 upper=3.0 effort=40 velocity=2.0
- added joint RF_ffe: type revolute, parent RF_shoulder, child RF_forearm, origin xyz=0 -0.2 0.025 rpy=0 0 0, axis 0 1 0, limit lower=-1.7 upper=0.5 effort=50 velocity=2.0
- added joint RF_haa: type revolute, parent base_fh, child RF_shoulder, origin xyz=0.35 -0.225 -0.23 rpy=0 0 0, axis 1 0 0, limit lower=-0.2 upper=0.2 effort=18 velocity=41
- added joint RF_hfe: type revolute, parent RF_pastern, child RF_hoof, origin xyz=0 0 -0.1, axis 0 1 0, limit lower=-0.3 upper=1.2 effort=20 velocity=2.0
- added joint RF_pfe: type revolute, parent RF_cannon, child RF_pastern, origin xyz=0.04 0 -0.32, axis 0 1 0, limit lower=-1.2 upper=0.5 effort=30 velocity=2.0

Commit message: using more realistic numbers (except for izz)

File: resources/robots/mini_horse/urdf/mini_horse_simple.urdf (robot description, URDF)
Before this commit: robot mini_horse, 22 links, 21 joints
Links:
- link LF_cannon: mass 1.0 -> 0.237
- link LF_forearm: mass 1.0 -> 4.795
- link LF_hoof: mass 0.2 -> 0.272
- link LF_pastern: mass 0.5 -> 0.912
- link LF_shoulder: mass 2.0 -> 4.795
- link LR_cannon: mass 1.0 -> 0.237
- link LR_forearm: mass 1.0 -> 4.795
- link LR_hoof: mass 0.2 -> 0.272
- link LR_pastern: mass 0.5 -> 0.912
- link LR_shoulder: mass 2.0 -> 4.795
- link RF_cannon: mass 1.0 -> 0.237
- link RF_forearm: mass 1.0 -> 4.795
- link RF_hoof: mass 0.2 -> 0.272
- link RF_pastern: mass 0.5 -> 0.912
- link RF_shoulder: mass 2.0 -> 4.795
- link RR_cannon: mass 1.0 -> 0.237
- link RR_forearm: mass 1.0 -> 4.795
- link RR_hoof: mass 0.2 -> 0.272
- link RR_pastern: mass 0.5 -> 0.912
- link RR_shoulder: mass 2.0 -> 4.795
- link base_bh: mass 4.0 -> 145.0
- link base_fh: mass 8.0 -> 345.0
