Commit message: mini_cheetah with horse mass

File: resources/robots/mini_cheetah/urdf/mini_cheetah_simple.urdf (robot description, URDF)
Before this commit: robot mini_cheetah, 17 links, 16 joints
Links:
- link base: mass 3.3 -> 490
- link lf_foot: mass 0.01 -> 0.20
- link lf_hip: mass 0.54 -> 4.558
- link lf_shank: mass 0.064 -> 2.02
- link lf_thigh: mass 0.634 -> 4.558
- link lh_foot: mass 0.01 -> 0.20
- link lh_hip: mass 0.54 -> 4.558
- link lh_shank: mass 0.064 -> 2.02
- link lh_thigh: mass 0.634 -> 4.558
- link rf_foot: mass 0.01 -> 0.20
- link rf_hip: mass 0.54 -> 4.558
- link rf_shank: mass 0.064 -> 2.02
- link rf_thigh: mass 0.634 -> 4.558
- link rh_foot: mass 0.01 -> 0.20
- link rh_hip: mass 0.54 -> 4.558
- link rh_shank: mass 0.064 -> 2.02
- link rh_thigh: mass 0.634 -> 4.558
Joints:
- joint 1_rf_haa: limit lower=-1.5 upper=1.5 effort=18 velocity=41 -> lower=-1.5 upper=1.5 effort=164 velocity=41
- joint 2_lf_haa: limit lower=-1.5 upper=1.5 effort=18 velocity=41 -> lower=-1.5 upper=1.5 effort=164 velocity=41
- joint 3_rh_haa: limit lower=-1.5 upper=1.5 effort=18 velocity=41 -> lower=-1.5 upper=1.5 effort=164 velocity=41
- joint 4_lh_haa: limit lower=-1.5 upper=1.5 effort=18 velocity=41 -> lower=-1.5 upper=1.5 effort=164 velocity=41
- joint lf_hfe: limit lower=-2.6 upper=2.6 effort=18 velocity=41 -> lower=-2.6 upper=2.6 effort=172 velocity=41
- joint lf_kfe: limit lower=-2.7 upper=2.7 effort=28 velocity=26.8 -> lower=-2.7 upper=2.7 effort=840 velocity=26.8
- joint lh_hfe: limit lower=-2.6 upper=2.6 effort=18 velocity=41 -> lower=-2.6 upper=2.6 effort=172 velocity=41
- joint lh_kfe: limit lower=-2.7 upper=2.7 effort=28 velocity=26.8 -> lower=-2.7 upper=2.7 effort=840 velocity=26.8
- joint rf_hfe: limit lower=-2.6 upper=2.6 effort=18 velocity=41 -> lower=-2.6 upper=2.6 effort=172 velocity=41
- joint rf_kfe: limit lower=-2.7 upper=2.7 effort=28 velocity=26.8 -> lower=-2.7 upper=2.7 effort=840 velocity=26.8
- joint rh_hfe: limit lower=-2.6 upper=2.6 effort=18 velocity=41 -> lower=-2.6 upper=2.6 effort=172 velocity=41
- joint rh_kfe: limit lower=-2.7 upper=2.7 effort=28 velocity=26.8 -> lower=-2.7 upper=2.7 effort=840 velocity=26.8

Commit message: scale inertia

File: resources/robots/mini_cheetah/urdf/mini_cheetah_simple.urdf (robot description, URDF)
Before this commit: robot mini_cheetah, 17 links, 16 joints
Links:
- link lf_shank: geometry visual mesh filename=meshes/lower_leg.dae
- link lf_thigh: geometry visual mesh filename=meshes/mini_vision_upper_leg.dae
- link lh_shank: geometry visual mesh filename=meshes/lower_leg.dae
- link lh_thigh: geometry visual mesh filename=meshes/mini_vision_upper_leg.dae
- link rh_shank: geometry visual mesh filename=meshes/lower_leg.dae
- link rh_thigh: geometry visual mesh filename=meshes/mini_vision_upper_leg.dae
Joints:
- joint 1_rf_haa: limit lower=-1.5 upper=1.5 effort=164 velocity=41 -> lower=-1.5 upper=1.5 effort=309 velocity=41
- joint 2_lf_haa: limit lower=-1.5 upper=1.5 effort=164 velocity=41 -> lower=-1.5 upper=1.5 effort=309 velocity=41
- joint 3_rh_haa: limit lower=-1.5 upper=1.5 effort=164 velocity=41 -> lower=-1.5 upper=1.5 effort=309 velocity=41
- joint 4_lh_haa: limit lower=-1.5 upper=1.5 effort=164 velocity=41 -> lower=-1.5 upper=1.5 effort=309 velocity=41
- joint lf_hfe: limit lower=-2.6 upper=2.6 effort=172 velocity=41 -> lower=-2.6 upper=2.6 effort=250 velocity=41
- joint lf_kfe: limit lower=-2.7 upper=2.7 effort=840 velocity=26.8 -> lower=-2.7 upper=2.7 effort=2793 velocity=26.8
- joint lh_hfe: limit lower=-2.6 upper=2.6 effort=172 velocity=41 -> lower=-2.6 upper=2.6 effort=250 velocity=41
- joint lh_kfe: limit lower=-2.7 upper=2.7 effort=840 velocity=26.8 -> lower=-2.7 upper=2.7 effort=2793 velocity=26.8
- joint rf_hfe: limit lower=-2.6 upper=2.6 effort=172 velocity=41 -> lower=-2.6 upper=2.6 effort=250 velocity=41
- joint rf_kfe: limit lower=-2.7 upper=2.7 effort=840 velocity=26.8 -> lower=-2.7 upper=2.7 effort=2793 velocity=26.8
- joint rh_hfe: limit lower=-2.6 upper=2.6 effort=172 velocity=41 -> lower=-2.6 upper=2.6 effort=250 velocity=41
- joint rh_kfe: limit lower=-2.7 upper=2.7 effort=840 velocity=26.8 -> lower=-2.7 upper=2.7 effort=2793 velocity=26.8

Commit message: baseline - split body

File: resources/robots/mini_cheetah/urdf/mini_cheetah_simple.urdf (robot description, URDF)
Before this commit: robot mini_cheetah, 17 links, 16 joints
Links:
- removed link base
- added link back_base, mass 145; collision box size=0.10 0.20 0.10; visual box size=0.10 0.20 0.10
- added link front_base, mass 345; collision box size=0.20 0.20 0.10; visual box size=0.20 0.20 0.10
Joints:
- added joint base_joint: type revolute, parent front_base, child back_base, origin xyz=-0.10 0 0.05 rpy=0 0 0, axis 0 1 0, limit lower=-0.2 upper=0.2 effort=18 velocity=41
- joint 1_rf_haa: parent base -> front_base
- joint 2_lf_haa: parent base -> front_base
- joint 3_rh_haa: origin xyz=-0.14775 -0.049 0.0 rpy=0 3.141592 0 -> xyz=-0.14775 -0.049 -0.05 rpy=0 3.141592 0; parent base -> back_base
- joint 4_lh_haa: origin xyz=-0.14775 0.049 0.0 rpy=0 3.141592 0 -> xyz=-0.14775 0.049 -0.05 rpy=0 3.141592 0; parent base -> back_base

Commit message: mini_cheetah with horse values

File: resources/robots/mini_cheetah/urdf/mini_cheetah_simple.urdf (robot description, URDF)
Before this commit: robot mini_cheetah, 18 links, 17 joints
Links:
- added link lf_pastern, mass 0.875; collision box size=0.06 0.06 0.08; visual cylinder length=0.13 radius=0.03
- added link lh_pastern, mass 0.875; collision box size=0.06 0.06 0.12; visual cylinder length=0.15 radius=0.03
- added link rf_pastern, mass 0.875; collision box size=0.06 0.06 0.08; visual cylinder length=0.13 radius=0.03
- added link rh_pastern, mass 0.875; collision box size=0.06 0.06 0.12; visual cylinder length=0.15 radius=0.03
- link back_base: geometry collision box size=0.41 0.38 0.51; visual box size=0.51 0.38 0.61
- link front_base: geometry collision box size=1.02 0.38 0.51; visual box size=1.02 0.38 0.61
- link lf_foot: geometry collision box size=0.1 0.1 0.05; visual cylinder length=0.08 radius=0.05
- link lf_hip: geometry visual cylinder length=0.05 radius=0.075
- link lf_shank: geometry collision box size=0.08 0.08 0.25; visual cylinder length=0.3 radius=0.04
- link lf_thigh: geometry collision box size=0.15 0.15 0.4; visual cylinder length=0.46 radius=0.075
- link lh_foot: geometry collision box size=0.1 0.1 0.05; visual cylinder length=0.08 radius=0.05
- link lh_hip: geometry visual cylinder length=0.05 radius=0.075
- link lh_shank: geometry collision box size=0.1 0.1 0.3; visual cylinder length=0.36 radius=0.05
- link lh_thigh: geometry collision box size=0.175 0.175 0.4; visual cylinder length=0.46 radius=0.09
- link rf_foot: geometry collision box size=0.1 0.1 0.05; visual cylinder length=0.08 radius=0.05
- link rf_hip: geometry visual cylinder length=0.05 radius=0.075
- link rf_shank: geometry collision box size=0.08 0.08 0.25; visual cylinder length=0.3 radius=0.04
- link rf_thigh: geometry collision box size=0.15 0.15 0.4; visual cylinder length=0.46 radius=0.075
- link rh_foot: geometry collision box size=0.1 0.1 0.05; visual cylinder length=0.08 radius=0.05
- link rh_hip: geometry visual cylinder length=0.05 radius=0.075
- link rh_shank: geometry collision box size=0.1 0.1 0.3; visual cylinder length=0.36 radius=0.05
- link rh_thigh: geometry collision box size=0.175 0.175 0.4; visual cylinder length=0.46 radius=0.09
Joints:
- removed joint lf_shank_to_foot
- removed joint lh_shank_to_foot
- removed joint rf_shank_to_foot
- removed joint rh_shank_to_foot
- added joint lf_pastern_to_foot: type revolute, parent lf_pastern, child lf_foot, origin xyz=0.0 0.0 -0.15 rpy=0.0 0.0 0.0, axis 0 -1 0, limit lower=-1.0 upper=0.3 effort=20 velocity=2.0
- added joint lf_pfe: type revolute, parent lf_shank, child lf_pastern, origin xyz=0.05 0.0 -0.3 rpy=0.0 0 0.0, axis 0 -1 0, limit lower=-1.2 upper=0.5 effort=2793 velocity=26.8
- added joint lh_pastern_to_foot: type revolute, parent lh_pastern, child lh_foot, origin xyz=0.0 0.0 -0.16 rpy=0.0 0.0 0.0, axis 0 -1 0, limit lower=-1.0 upper=0.3 effort=20 velocity=2.0
- added joint lh_pfe: type revolute, parent lh_shank, child lh_pastern, origin xyz=-0.045 0.0 -0.39 rpy=0.0 0 0.0, axis 0 -1 0, limit lower=-1.0 upper=0.0 effort=2793 velocity=26.8
- added joint rf_pastern_to_foot: type revolute, parent rf_pastern, child rf_foot, origin xyz=0.0 0.0 -0.15 rpy=0.0 0.0 0.0, axis 0 -1 0, limit lower=-1.0 upper=0.3 effort=20 velocity=2.0
- added joint rf_pfe: type revolute, parent rf_shank, child rf_pastern, origin xyz=0.05 0.0 -0.3 rpy=0.0 0 0.0, axis 0 -1 0, limit lower=-1.2 upper=0.5 effort=2793 velocity=26.8
- added joint rh_pastern_to_foot: type revolute, parent rh_pastern, child rh_foot, origin xyz=0.0 0.0 -0.16 rpy=0.0 0.0 0.0, axis 0 -1 0, limit lower=-1.0 upper=0.3 effort=20 velocity=2.0
- added joint rh_pfe: type revolute, parent rh_shank, child rh_pastern, origin xyz=-0.045 0.0 -0.39 rpy=0.0 0 0.0, axis 0 -1 0, limit lower=-1.0 upper=0.0 effort=2793 velocity=26.8
- joint 1_rf_haa: limit lower=-1.5 upper=1.5 effort=309 velocity=41 -> upper=0.2 effort=309 velocity=41; origin xyz=0.14775 -0.049 0.0 rpy=0 0 0 -> xyz=0.35 -0.225 -0.23 rpy=0 0 0
- joint 2_lf_haa: limit lower=-1.5 upper=1.5 effort=309 velocity=41 -> lower=-0.2 upper=0.2 effort=309 velocity=41; origin xyz=0.14775 0.049 0.0 rpy=0 0 0 -> xyz=0.35 0.225 -0.23 rpy=0 0 0
- joint 3_rh_haa: limit lower=-1.5 upper=1.5 effort=309 velocity=41 -> lower=-0.2 upper=0.2 effort=309 velocity=41; origin xyz=-0.14775 -0.049 -0.05 rpy=0 3.141592 0 -> xyz=-0.3 -0.225 -0.43 rpy=0 3.141592 0
- joint 4_lh_haa: limit lower=-1.5 upper=1.5 effort=309 velocity=41 -> lower=-0.2 upper=0.2 effort=309 velocity=41; origin xyz=-0.14775 0.049 -0.05 rpy=0 3.141592 0 -> xyz=-0.3 0.225 -0.43 rpy=0 3.141592 0
- joint base_joint: limit lower=-0.2 upper=0.2 effort=18 velocity=41 -> lower=-0.2 upper=0.2 effort=1100 velocity=41; origin xyz=-0.10 0 0.05 rpy=0 0 0 -> xyz=-0.5 0 0.3 rpy=0 0 0
- joint lf_hfe: axis 0 -1 0 -> 0 1 0; limit lower=-2.6 upper=2.6 effort=250 velocity=41 -> lower=-1.5 upper=0.5 effort=250 velocity=41; origin xyz=0.055 0.019 0.00 rpy=0.0 0.0 0.0 -> xyz=0.0 0.12 -0.05 rpy=0.0 0.0 0.0
- joint lf_kfe: limit lower=-2.7 upper=2.7 effort=2793 velocity=26.8 -> lower=-3.0 upper=0.0 effort=2793 velocity=26.8; origin xyz=0.0 0.049 -0.2085 rpy=0.0 0 0.0 -> xyz=-0.07 0.0 -0.43 rpy=0.0 0 0.0
- joint lh_hfe: axis 0 -1 0 -> 0 1 0; limit lower=-2.6 upper=2.6 effort=250 velocity=41 -> lower=-0.5 upper=1.5 effort=250 velocity=41; origin xyz=0.055 0.019 0.00 rpy=0.0 3.141592 0.0 -> xyz=0.0 0.12 -0.05 rpy=0.0 3.141592 0.0
- joint lh_kfe: limit lower=-2.7 upper=2.7 effort=2793 velocity=26.8 -> lower=0.0 upper=3.0 effort=2793 velocity=26.8; origin xyz=0.0 0.049 -0.2085 rpy=0.0 0 0.0 -> xyz=0.09 0.0 -0.51 rpy=0.0 0 0.0
- joint rf_hfe: limit lower=-2.6 upper=2.6 effort=250 velocity=41 -> lower=-0.5 upper=1.7 effort=250 velocity=41; origin xyz=0.055 -0.019 0.00 rpy=0.0 0.0 0.0 -> xyz=0.0 -0.12 -0.05 rpy=0.0 0.0 0.0
- joint rf_kfe: limit lower=-2.7 upper=2.7 effort=2793 velocity=26.8 -> lower=-3.0 upper=0.0 effort=2793 velocity=26.8; origin xyz=0.0 -0.049 -0.2085 rpy=0.0 0 0.0 -> xyz=-0.07 0.0 -0.43 rpy=0.0 0 0.0
- joint rh_hfe: limit lower=-2.6 upper=2.6 effort=250 velocity=41 -> lower=-1.5 upper=0.5 effort=250 velocity=41; origin xyz=0.055 -0.019 0.00 rpy=0.0 3.141592 0.0 -> xyz=0.0 -0.12 -0.05 rpy=0.0 3.141592 0.0
- joint rh_kfe: limit lower=-2.7 upper=2.7 effort=2793 velocity=26.8 -> lower=0.0 upper=3.0 effort=2793 velocity=26.8; origin xyz=0.0 -0.049 -0.2085 rpy=0.0 0 0.0 -> xyz=0.09 0.0 -0.51 rpy=0.0 0 0.0

Commit message: stable horse but can't stand

File: resources/robots/mini_cheetah/urdf/mini_cheetah_simple.urdf (robot description, URDF)
Before this commit: robot mini_cheetah, 22 links, 21 joints
Links:
- link lf_shank: mass 2.02 -> 1.404
- link lh_shank: mass 2.02 -> 1.404
- link rf_shank: mass 2.02 -> 1.404
- link rh_shank: mass 2.02 -> 1.404
Joints:
- joint 1_rf_haa: limit upper=0.2 effort=309 velocity=41 -> lower=-0.2 upper=0.2 effort=35500 velocity=41
- joint 2_lf_haa: limit lower=-0.2 upper=0.2 effort=309 velocity=41 -> lower=-0.2 upper=0.2 effort=35500 velocity=41
- joint 3_rh_haa: limit lower=-0.2 upper=0.2 effort=309 velocity=41 -> lower=-0.2 upper=0.2 effort=35500 velocity=41
- joint 4_lh_haa: limit lower=-0.2 upper=0.2 effort=309 velocity=41 -> lower=-0.2 upper=0.2 effort=35500 velocity=41
- joint lf_hfe: limit lower=-1.5 upper=0.5 effort=250 velocity=41 -> lower=-1.5 upper=0.5 effort=400000 velocity=41
- joint lf_kfe: limit lower=-3.0 upper=0.0 effort=2793 velocity=26.8 -> lower=-3.0 upper=0.0 effort=400000 velocity=26.8
- joint lf_pastern_to_foot: limit lower=-1.0 upper=0.3 effort=20 velocity=2.0 -> lower=-1.0 upper=0.3 effort=2793 velocity=2.0
- joint lf_pfe: limit lower=-1.2 upper=0.5 effort=2793 velocity=26.8 -> lower=-1.2 upper=0.5 effort=4000 velocity=26.8
- joint lh_hfe: limit lower=-0.5 upper=1.5 effort=250 velocity=41 -> lower=-0.5 upper=1.5 effort=400000 velocity=41
- joint lh_kfe: limit lower=0.0 upper=3.0 effort=2793 velocity=26.8 -> lower=0.0 upper=3.0 effort=400000 velocity=26.8
- joint lh_pastern_to_foot: limit lower=-1.0 upper=0.3 effort=20 velocity=2.0 -> lower=-1.0 upper=0.3 effort=2793 velocity=2.0
- joint lh_pfe: limit lower=-1.0 upper=0.0 effort=2793 velocity=26.8 -> lower=-1.0 upper=0.0 effort=4000 velocity=26.8
- joint rf_hfe: limit lower=-0.5 upper=1.7 effort=250 velocity=41 -> lower=-0.5 upper=1.7 effort=400000 velocity=41
- joint rf_kfe: limit lower=-3.0 upper=0.0 effort=2793 velocity=26.8 -> lower=-3.0 upper=0.0 effort=400000 velocity=26.8
- joint rf_pastern_to_foot: limit lower=-1.0 upper=0.3 effort=20 velocity=2.0 -> lower=-1.0 upper=0.3 effort=2793 velocity=2.0
- joint rf_pfe: limit lower=-1.2 upper=0.5 effort=2793 velocity=26.8 -> lower=-1.2 upper=0.5 effort=4000 velocity=26.8
- joint rh_hfe: limit lower=-1.5 upper=0.5 effort=250 velocity=41 -> lower=-1.5 upper=0.5 effort=400000 velocity=41
- joint rh_kfe: limit lower=0.0 upper=3.0 effort=2793 velocity=26.8 -> lower=0.0 upper=3.0 effort=400000 velocity=26.8
- joint rh_pastern_to_foot: limit lower=-1.0 upper=0.3 effort=20 velocity=2.0 -> lower=-1.0 upper=0.3 effort=2793 velocity=2.0
- joint rh_pfe: limit lower=-1.0 upper=0.0 effort=2793 velocity=26.8 -> lower=-1.0 upper=0.0 effort=4000 velocity=26.8

Commit message: realistic effort values

File: resources/robots/mini_cheetah/urdf/mini_cheetah_simple.urdf (robot description, URDF)
Before this commit: robot mini_cheetah, 22 links, 21 joints
Joints:
- joint 1_rf_haa: limit lower=-0.2 upper=0.2 effort=35500 velocity=41 -> lower=-0.2 upper=0.2 effort=800 velocity=41
- joint 2_lf_haa: limit lower=-0.2 upper=0.2 effort=35500 velocity=41 -> lower=-0.2 upper=0.2 effort=800 velocity=41
- joint 3_rh_haa: limit lower=-0.2 upper=0.2 effort=35500 velocity=41 -> lower=-0.2 upper=0.2 effort=800 velocity=41
- joint 4_lh_haa: limit lower=-0.2 upper=0.2 effort=35500 velocity=41 -> lower=-0.2 upper=0.2 effort=800 velocity=41
- joint lf_hfe: limit lower=-1.5 upper=0.5 effort=400000 velocity=41 -> lower=-1.5 upper=0.5 effort=700 velocity=41
- joint lf_kfe: limit lower=-3.0 upper=0.0 effort=400000 velocity=26.8 -> lower=-3.0 upper=0.0 effort=600 velocity=26.8
- joint lf_pastern_to_foot: limit lower=-1.0 upper=0.3 effort=2793 velocity=2.0 -> lower=-1.0 upper=0.3 effort=300 velocity=2.0
- joint lf_pfe: limit lower=-1.2 upper=0.5 effort=4000 velocity=26.8 -> lower=-1.2 upper=0.5 effort=500 velocity=26.8
- joint lh_hfe: limit lower=-0.5 upper=1.5 effort=400000 velocity=41 -> lower=-0.5 upper=1.5 effort=700 velocity=41
- joint lh_kfe: limit lower=0.0 upper=3.0 effort=400000 velocity=26.8 -> lower=0.0 upper=3.0 effort=600 velocity=26.8
- joint lh_pastern_to_foot: limit lower=-1.0 upper=0.3 effort=2793 velocity=2.0 -> lower=-1.0 upper=0.3 effort=300 velocity=2.0
- joint lh_pfe: limit lower=-1.0 upper=0.0 effort=4000 velocity=26.8 -> lower=-1.0 upper=0.0 effort=500 velocity=26.8
- joint rf_hfe: limit lower=-0.5 upper=1.7 effort=400000 velocity=41 -> lower=-0.5 upper=1.7 effort=700 velocity=41
- joint rf_kfe: limit lower=-3.0 upper=0.0 effort=400000 velocity=26.8 -> lower=-3.0 upper=0.0 effort=600 velocity=26.8
- joint rf_pastern_to_foot: limit lower=-1.0 upper=0.3 effort=2793 velocity=2.0 -> lower=-1.0 upper=0.3 effort=300 velocity=2.0
- joint rf_pfe: limit lower=-1.2 upper=0.5 effort=4000 velocity=26.8 -> lower=-1.2 upper=0.5 effort=500 velocity=26.8
- joint rh_hfe: limit lower=-1.5 upper=0.5 effort=400000 velocity=41 -> lower=-1.5 upper=0.5 effort=700 velocity=41
- joint rh_kfe: limit lower=0.0 upper=3.0 effort=400000 velocity=26.8 -> lower=0.0 upper=3.0 effort=600 velocity=26.8
- joint rh_pastern_to_foot: limit lower=-1.0 upper=0.3 effort=2793 velocity=2.0 -> lower=-1.0 upper=0.3 effort=300 velocity=2.0
- joint rh_pfe: limit lower=-1.0 upper=0.0 effort=4000 velocity=26.8 -> lower=-1.0 upper=0.0 effort=500 velocity=26.8

Commit message: better results

File: resources/robots/mini_cheetah/urdf/mini_cheetah_simple.urdf (robot description, URDF)
Before this commit: robot mini_cheetah, 22 links, 21 joints
Joints:
- joint 1_rf_haa: limit lower=-0.2 upper=0.2 effort=800 velocity=41 -> lower=-0.2 upper=0.2 effort=1000 velocity=41
- joint 2_lf_haa: limit lower=-0.2 upper=0.2 effort=800 velocity=41 -> lower=-0.2 upper=0.2 effort=1000 velocity=41
- joint 3_rh_haa: limit lower=-0.2 upper=0.2 effort=800 velocity=41 -> lower=-0.2 upper=0.2 effort=1000 velocity=41
- joint 4_lh_haa: limit lower=-0.2 upper=0.2 effort=800 velocity=41 -> lower=-0.2 upper=0.2 effort=1000 velocity=41
- joint lf_kfe: limit lower=-3.0 upper=0.0 effort=600 velocity=26.8 -> lower=-3.0 upper=0.0 effort=1000 velocity=26.8
- joint lh_kfe: limit lower=0.0 upper=3.0 effort=600 velocity=26.8 -> lower=0.0 upper=3.0 effort=1000 velocity=26.8
- joint rf_kfe: limit lower=-3.0 upper=0.0 effort=600 velocity=26.8 -> lower=-3.0 upper=0.0 effort=1000 velocity=26.8
- joint rh_kfe: limit lower=0.0 upper=3.0 effort=600 velocity=26.8 -> lower=0.0 upper=3.0 effort=1000 velocity=26.8

Commit message: manual merge of non-logging part of yl/horse_RL

File: resources/robots/mini_cheetah/urdf/mini_cheetah_simple.urdf (robot description, URDF)
Before this commit: robot mini_cheetah, 22 links, 21 joints
Joints:
- joint 1_rf_haa: limit lower=-0.2 upper=0.2 effort=35500 velocity=41 -> lower=-0.2 upper=0.2 effort=1000 velocity=41
- joint 2_lf_haa: limit lower=-0.2 upper=0.2 effort=35500 velocity=41 -> lower=-0.2 upper=0.2 effort=1000 velocity=41
- joint 3_rh_haa: limit lower=-0.2 upper=0.2 effort=35500 velocity=41 -> lower=-0.2 upper=0.2 effort=1000 velocity=41
- joint 4_lh_haa: limit lower=-0.2 upper=0.2 effort=35500 velocity=41 -> lower=-0.2 upper=0.2 effort=1000 velocity=41
- joint lf_hfe: limit lower=-1.5 upper=0.5 effort=400000 velocity=41 -> lower=-1.5 upper=0.5 effort=700 velocity=41
- joint lf_kfe: limit lower=-3.0 upper=0.0 effort=400000 velocity=26.8 -> lower=-3.0 upper=0.0 effort=1000 velocity=26.8
- joint lf_pastern_to_foot: limit lower=-1.0 upper=0.3 effort=2793 velocity=2.0 -> lower=-1.0 upper=0.3 effort=300 velocity=2.0
- joint lf_pfe: limit lower=-1.2 upper=0.5 effort=4000 velocity=26.8 -> lower=-1.2 upper=0.5 effort=500 velocity=26.8
- joint lh_hfe: limit lower=-0.5 upper=1.5 effort=400000 velocity=41 -> lower=-0.5 upper=1.5 effort=700 velocity=41
- joint lh_kfe: limit lower=0.0 upper=3.0 effort=400000 velocity=26.8 -> lower=0.0 upper=3.0 effort=1000 velocity=26.8
- joint lh_pastern_to_foot: limit lower=-1.0 upper=0.3 effort=2793 velocity=2.0 -> lower=-1.0 upper=0.3 effort=300 velocity=2.0
- joint lh_pfe: limit lower=-1.0 upper=0.0 effort=4000 velocity=26.8 -> lower=-1.0 upper=0.0 effort=500 velocity=26.8
- joint rf_hfe: limit lower=-0.5 upper=1.7 effort=400000 velocity=41 -> lower=-0.5 upper=1.7 effort=700 velocity=41
- joint rf_kfe: limit lower=-3.0 upper=0.0 effort=400000 velocity=26.8 -> lower=-3.0 upper=0.0 effort=1000 velocity=26.8
- joint rf_pastern_to_foot: limit lower=-1.0 upper=0.3 effort=2793 velocity=2.0 -> lower=-1.0 upper=0.3 effort=300 velocity=2.0
- joint rf_pfe: limit lower=-1.2 upper=0.5 effort=4000 velocity=26.8 -> lower=-1.2 upper=0.5 effort=500 velocity=26.8
- joint rh_hfe: limit lower=-1.5 upper=0.5 effort=400000 velocity=41 -> lower=-1.5 upper=0.5 effort=700 velocity=41
- joint rh_kfe: limit lower=0.0 upper=3.0 effort=400000 velocity=26.8 -> lower=0.0 upper=3.0 effort=1000 velocity=26.8
- joint rh_pastern_to_foot: limit lower=-1.0 upper=0.3 effort=2793 velocity=2.0 -> lower=-1.0 upper=0.3 effort=300 velocity=2.0
- joint rh_pfe: limit lower=-1.0 upper=0.0 effort=4000 velocity=26.8 -> lower=-1.0 upper=0.0 effort=500 velocity=26.8
