Commit message: WIP: partial urdf changes

File: resources/robots/mini_cheetah/urdf/mini_cheetah_simple.urdf (robot description, URDF)
Before this commit: robot mini_cheetah, 22 links, 21 joints
Links:
- removed link lf_foot
- removed link lf_hip
- removed link lf_pastern
- removed link lf_shank
- removed link lf_thigh
- removed link lh_foot
- removed link lh_hip
- removed link lh_pastern
- removed link lh_shank
- removed link lh_thigh
- removed link rf_foot
- removed link rf_hip
- removed link rf_pastern
- removed link rf_shank
- removed link rf_thigh
- removed link rh_foot
- removed link rh_hip
- removed link rh_pastern
- removed link rh_shank
- removed link rh_thigh
- added link fl_foot, mass 0.20; collision box size=0.1 0.1 0.05; visual cylinder length=0.08 radius=0.05
- added link fl_hip, mass 4.558; visual cylinder length=0.05 radius=0.075
- added link fl_pastern, mass 0.875; collision box size=0.06 0.06 0.08; visual cylinder length=0.13 radius=0.03
- added link fl_shank, mass 1.404; collision box size=0.08 0.08 0.25; visual cylinder length=0.3 radius=0.04
- added link fl_thigh, mass 4.558; collision box size=0.15 0.15 0.3; visual cylinder length=0.3 radius=0.075
- added link fr_foot, mass 0.20; collision box size=0.1 0.1 0.05; visual cylinder length=0.08 radius=0.05
- added link fr_hip, mass 4.558; visual cylinder length=0.05 radius=0.075
- added link fr_pastern, mass 0.875; collision box size=0.06 0.06 0.08; visual cylinder length=0.13 radius=0.03
- added link fr_shank, mass 1.404; collision box size=0.08 0.08 0.25; visual cylinder length=0.3 radius=0.04
- added link fr_thigh, mass 4.558; collision box size=0.15 0.15 0.4; visual cylinder length=0.46 radius=0.075
- added link hl_foot, mass 0.20; collision box size=0.1 0.1 0.05; visual cylinder length=0.08 radius=0.05
- added link hl_hip, mass 4.558; visual cylinder length=0.05 radius=0.075
- added link hl_pastern, mass 0.875; collision box size=0.06 0.06 0.12; visual cylinder length=0.15 radius=0.03
- added link hl_shank, mass 1.404; collision box size=0.1 0.1 0.3; visual cylinder length=0.36 radius=0.05
- added link hl_thigh, mass 4.558; collision box size=0.175 0.175 0.4; visual cylinder length=0.46 radius=0.09
- added link hr_foot, mass 0.20; collision box size=0.1 0.1 0.05; visual cylinder length=0.08 radius=0.05
- added link hr_hip, mass 4.558; visual cylinder length=0.05 radius=0.075
- added link hr_pastern, mass 0.875; collision box size=0.06 0.06 0.12; visual cylinder length=0.15 radius=0.03
- added link hr_shank, mass 1.404; collision box size=0.1 0.1 0.3; visual cylinder length=0.36 radius=0.05
- added link hr_thigh, mass 4.558; collision box size=0.175 0.175 0.4; visual cylinder length=0.46 radius=0.09
Joints:
- removed joint 1_rf_haa
- removed joint 2_lf_haa
- removed joint 3_rh_haa
- removed joint 4_lh_haa
- removed joint lf_hfe
- removed joint lf_kfe
- removed joint lf_pastern_to_foot
- removed joint lf_pfe
- removed joint lh_hfe
- removed joint lh_kfe
- removed joint lh_pastern_to_foot
- removed joint lh_pfe
- removed joint rf_hfe
- removed joint rf_kfe
- removed joint rf_pastern_to_foot
- removed joint rf_pfe
- removed joint rh_hfe
- removed joint rh_kfe
- removed joint rh_pastern_to_foot
- removed joint rh_pfe
- added joint 1_fr_haa: type revolute, parent front_base, child fr_hip, origin xyz=0.35 -0.225 -0.23 rpy=0 0 0, axis 1 0 0, limit lower=-0.2 upper=0.2 effort=1000 velocity=41
- added joint 2_fl_haa: type revolute, parent front_base, child fl_hip, origin xyz=0.35 0.225 -0.23 rpy=0 0 0, axis 1 0 0, limit lower=-0.2 upper=0.2 effort=1000 velocity=41
- added joint 3_hr_haa: type revolute, parent back_base, child hr_hip, origin xyz=-0.3 -0.225 -0.3 rpy=0 3.141592 0, axis -1 0 0, limit lower=-0.2 upper=0.2 effort=1000 velocity=41
- added joint 4_hl_haa: type revolute, parent back_base, child hl_hip, origin xyz=-0.3 0.225 -0.3 rpy=0 3.141592 0, axis -1 0 0, limit lower=-0.2 upper=0.2 effort=1000 velocity=41
- added joint fl_hfe: type revolute, parent fl_hip, child fl_thigh, origin xyz=0.0 0.12 -0.05 rpy=0.0 0.6 0.0, axis 0 1 0, limit lower=-0.7 upper=0.6 effort=700 velocity=41
- added joint fl_kfe: type revolute, parent fl_thigh, child fl_shank, origin xyz=0.0 0.0 -0.3 rpy=0.0 -0.6 0.0, axis 0 1 0, limit lower=-1.6 upper=0.1 effort=1000 velocity=26.8
- added joint fl_pastern_to_foot: type revolute, parent fl_pastern, child fl_foot, origin xyz=0.0 0.0 -0.25 rpy=0.0 0.0 0.0, axis 0 1 0, limit lower=-0.3 upper=1.5 effort=300 velocity=2.0
- added joint fl_pfe: type revolute, parent fl_shank, child fl_pastern, origin xyz=0.05 0.0 -0.3 rpy=0.0 0 0.0, axis 0 1 0, limit lower=-0.3 upper=2.0 effort=500 velocity=26.8
- added joint fr_hfe: type revolute, parent fr_hip, child fr_thigh, origin xyz=0.0 -0.12 -0.05 rpy=0.0 0.0 0.0, axis 0 -1 0, limit lower=-0.5 upper=1.7 effort=700 velocity=41
- added joint fr_kfe: type revolute, parent fr_thigh, child fr_shank, origin xyz=-0.07 0.0 -0.43 rpy=0.0 0 0.0, axis 0 -1 0, limit lower=-3.0 upper=2.0 effort=1000 velocity=26.8
- added joint fr_pastern_to_foot: type revolute, parent fr_pastern, child fr_foot, origin xyz=0.0 0.0 -0.15 rpy=0.0 0.0 0.0, axis 0 -1 0, limit lower=-1.0 upper=0.3 effort=300 velocity=2.0
- added joint fr_pfe: type revolute, parent fr_shank, child fr_pastern, origin xyz=0.05 0.0 -0.3 rpy=0.0 0 0.0, axis 0 -1 0, limit lower=-1.2 upper=0.5 effort=500 velocity=26.8
- added joint hl_hfe: type revolute, parent hl_hip, child hl_thigh, origin xyz=0.0 0.12 -0.05 rpy=0.0 2.841592 0.0, axis 0 1 0, limit lower=-0.5 upper=1.5 effort=700 velocity=41
- added joint hl_kfe: type revolute, parent hl_thigh, child hl_shank, origin xyz=0.0 0.0 -0.61 rpy=0.0 0.65 0.0, axis 0 1 0, limit lower=-0.2 upper=1.5 effort=1000 velocity=26.8
- added joint hl_pastern_to_foot: type revolute, parent hl_pastern, child hl_foot, origin xyz=0.0 0.0 -0.16 rpy=0.0 0.0 0.0, axis 0 -1 0, limit lower=-1.0 upper=0.3 effort=300 velocity=2.0
- added joint hl_pfe: type revolute, parent hl_shank, child hl_pastern, origin xyz=-0.045 0.0 -0.39 rpy=0.0 -0.35 0.0, axis 0 1 0, limit lower=-0.3 upper=2.5 effort=500 velocity=26.8
- added joint hr_hfe: type revolute, parent hr_hip, child hr_thigh, origin xyz=0.0 -0.12 -0.05 rpy=0.0 3.141592 0.0, axis 0 1 0, limit lower=-0.5 upper=1.5 effort=700 velocity=41
- added joint hr_kfe: type revolute, parent hr_thigh, child hr_shank, origin xyz=0.09 0.0 -0.51 rpy=0.0 0 0.0, axis 0 1 0, limit lower=-0.2 upper=3.0 effort=1000 velocity=26.8
- added joint hr_pastern_to_foot: type revolute, parent hr_pastern, child hr_foot, origin xyz=0.0 0.0 -0.16 rpy=0.0 0.0 0.0, axis 0 -1 0, limit lower=-1.0 upper=0.3 effort=300 velocity=2.0
- added joint hr_pfe: type revolute, parent hr_shank, child hr_pastern, origin xyz=-0.045 0.0 -0.39 rpy=0.0 0 0.0, axis 0 -1 0, limit lower=-1.0 upper=2.0 effort=500 velocity=26.8

Commit message: fix left legs

File: resources/robots/mini_cheetah/urdf/mini_cheetah_simple.urdf (robot description, URDF)
Before this commit: robot mini_cheetah, 22 links, 21 joints
Links:
- link fl_foot: geometry collision cylinder length=0.04 radius=0.05; visual cylinder length=0.04 radius=0.05
- link fl_pastern: geometry collision cylinder length=0.2 radius=0.03; visual cylinder length=0.2 radius=0.03
- link fl_shank: geometry collision cylinder length=0.3 radius=0.04; visual cylinder length=0.3 radius=0.04
- link fl_thigh: geometry collision cylinder length=0.25 radius=0.075; visual cylinder length=0.25 radius=0.075
- link fr_hip: geometry collision cylinder length=0.05 radius=0.075; visual cylinder length=0.05 radius=0.075
- link fr_thigh: geometry collision cylinder length=0.46 radius=0.075; visual cylinder length=0.46 radius=0.075
- link hl_foot: geometry collision cylinder length=0.04 radius=0.05; visual cylinder length=0.04 radius=0.05
- link hl_pastern: geometry collision cylinder length=0.25 radius=0.03; visual cylinder length=0.25 radius=0.03
- link hl_shank: geometry collision cylinder length=0.25 radius=0.04; visual cylinder length=0.25 radius=0.04
- link hl_thigh: geometry collision cylinder length=0.2 radius=0.09; visual cylinder length=0.2 radius=0.09
Joints:
- joint 4_hl_haa: origin xyz=-0.3 0.225 -0.3 rpy=0 3.141592 0 -> xyz=-0.3 0.225 -0.4 rpy=0 3.141592 0
- joint fl_kfe: limit lower=-1.6 upper=0.1 effort=1000 velocity=26.8 -> lower=-1.3 upper=0.1 effort=1000 velocity=26.8; origin xyz=0.0 0.0 -0.3 rpy=0.0 -0.6 0.0 -> xyz=0.0 0.0 -0.45 rpy=0.0 -0.6 0.0
- joint fl_pastern_to_foot: limit lower=-0.3 upper=1.5 effort=300 velocity=2.0 -> lower=-0.3 upper=1.8 effort=300 velocity=2.0; origin xyz=0.0 0.0 -0.25 rpy=0.0 0.0 0.0 -> xyz=0.025 0.0 -0.3 rpy=0.0 0.0 0.0
- joint fl_pfe: limit lower=-0.3 upper=2.0 effort=500 velocity=26.8 -> lower=-0.3 upper=2.2 effort=500 velocity=26.8; origin xyz=0.05 0.0 -0.3 rpy=0.0 0 0.0 -> xyz=0.0 0.0 -0.3 rpy=0.05 0 0.0
- joint hl_hfe: limit lower=-0.5 upper=1.5 effort=700 velocity=41 -> lower=-0.7 upper=1.5 effort=700 velocity=41
- joint hl_kfe: limit lower=-0.2 upper=1.5 effort=1000 velocity=26.8 -> lower=-0.2 upper=0.8 effort=1000 velocity=26.8; origin xyz=0.0 0.0 -0.61 rpy=0.0 0.65 0.0 -> xyz=0.0 0.0 -0.5 rpy=0.0 0.65 0.0
- joint hl_pastern_to_foot: axis 0 -1 0 -> 0 1 0; limit lower=-1.0 upper=0.3 effort=300 velocity=2.0 -> lower=-0.3 upper=1.8 effort=300 velocity=2.0; origin xyz=0.0 0.0 -0.16 rpy=0.0 0.0 0.0 -> xyz=0.0 0.0 -0.35 rpy=0.0 0.0 0.0
- joint hl_pfe: origin xyz=-0.045 0.0 -0.39 rpy=0.0 -0.35 0.0 -> xyz=-0.045 0.0 -0.35 rpy=0.0 -0.35 0.0

Commit message: mirror left and right

File: resources/robots/mini_cheetah/urdf/mini_cheetah_simple.urdf (robot description, URDF)
Before this commit: robot mini_cheetah, 22 links, 21 joints
Links:
- link fr_foot: geometry collision cylinder length=0.04 radius=0.05; visual cylinder length=0.04 radius=0.05
- link fr_hip: geometry visual cylinder length=0.05 radius=0.075
- link fr_pastern: geometry collision cylinder length=0.2 radius=0.03; visual cylinder length=0.2 radius=0.03
- link fr_shank: geometry collision cylinder length=0.3 radius=0.04; visual cylinder length=0.3 radius=0.04
- link fr_thigh: geometry collision cylinder length=0.25 radius=0.075; visual cylinder length=0.25 radius=0.075
- link front_base: geometry collision box size=.8 0.38 0.51; visual box size=0.8 0.38 0.61
- link hr_foot: geometry collision cylinder length=0.04 radius=0.05; visual cylinder length=0.04 radius=0.05
- link hr_pastern: geometry collision cylinder length=0.25 radius=0.03; visual cylinder length=0.25 radius=0.03
- link hr_shank: geometry collision cylinder length=0.25 radius=0.04; visual cylinder length=0.25 radius=0.04
- link hr_thigh: geometry collision cylinder length=0.2 radius=0.09; visual cylinder length=0.2 radius=0.09
Joints:
- joint 1_fr_haa: axis 1 0 0 -> -1 0 0
- joint 3_hr_haa: axis -1 0 0 -> 1 0 0
- joint fr_hfe: axis 0 -1 0 -> 0 1 0; limit lower=-0.5 upper=1.7 effort=700 velocity=41 -> lower=-0.7 upper=0.6 effort=700 velocity=41; origin xyz=0.0 -0.12 -0.05 rpy=0.0 0.0 0.0 -> xyz=0.0 0.12 -0.05 rpy=0.0 0.6 0.0
- joint fr_kfe: axis 0 -1 0 -> 0 1 0; limit lower=-3.0 upper=2.0 effort=1000 velocity=26.8 -> lower=-1.3 upper=0.1 effort=1000 velocity=26.8; origin xyz=-0.07 0.0 -0.43 rpy=0.0 0 0.0 -> xyz=0.0 0.0 -0.45 rpy=0.0 -0.6 0.0
- joint fr_pastern_to_foot: axis 0 -1 0 -> 0 1 0; limit lower=-1.0 upper=0.3 effort=300 velocity=2.0 -> lower=-0.3 upper=1.8 effort=300 velocity=2.0; origin xyz=0.0 0.0 -0.15 rpy=0.0 0.0 0.0 -> xyz=0.025 0.0 -0.3 rpy=0.0 0.0 0.0
- joint fr_pfe: axis 0 -1 0 -> 0 1 0; limit lower=-1.2 upper=0.5 effort=500 velocity=26.8 -> lower=-0.3 upper=2.2 effort=500 velocity=26.8; origin xyz=0.05 0.0 -0.3 rpy=0.0 0 0.0 -> xyz=0.0 0.0 -0.3 rpy=0.05 0 0.0
- joint hr_hfe: limit lower=-0.5 upper=1.5 effort=700 velocity=41 -> lower=-0.7 upper=1.5 effort=700 velocity=41; origin xyz=0.0 -0.12 -0.05 rpy=0.0 3.141592 0.0 -> xyz=0.0 0.12 -0.05 rpy=0.0 2.841592 0.0
- joint hr_kfe: limit lower=-0.2 upper=3.0 effort=1000 velocity=26.8 -> lower=-0.2 upper=0.8 effort=1000 velocity=26.8; origin xyz=0.09 0.0 -0.51 rpy=0.0 0 0.0 -> xyz=0.0 0.0 -0.5 rpy=0.0 0.65 0.0
- joint hr_pastern_to_foot: axis 0 -1 0 -> 0 1 0; limit lower=-1.0 upper=0.3 effort=300 velocity=2.0 -> lower=-0.3 upper=1.8 effort=300 velocity=2.0; origin xyz=0.0 0.0 -0.16 rpy=0.0 0.0 0.0 -> xyz=0.0 0.0 -0.35 rpy=0.0 0.0 0.0
- joint hr_pfe: axis 0 -1 0 -> 0 1 0; limit lower=-1.0 upper=2.0 effort=500 velocity=26.8 -> lower=-0.3 upper=2.5 effort=500 velocity=26.8; origin xyz=-0.045 0.0 -0.39 rpy=0.0 0 0.0 -> xyz=-0.045 0.0 -0.35 rpy=0.0 -0.35 0.0

Commit message: remove inertial offsets along y for symmetry

File: resources/robots/mini_cheetah/urdf/mini_cheetah_simple.urdf (robot description, URDF)
Before this commit: robot mini_cheetah, 22 links, 21 joints
Joints:
- joint 3_hr_haa: origin xyz=-0.3 -0.225 -0.3 rpy=0 3.141592 0 -> xyz=-0.3 -0.225 -0.4 rpy=0 3.141592 0
- joint fr_hfe: origin xyz=0.0 0.12 -0.05 rpy=0.0 0.6 0.0 -> xyz=0.0 -0.12 -0.05 rpy=0.0 0.6 0.0
- joint hr_hfe: origin xyz=0.0 0.12 -0.05 rpy=0.0 2.841592 0.0 -> xyz=0.0 -0.12 -0.05 rpy=0.0 2.841592 0.0

Commit message: rename urdf for symmetry ease, some minor tweaks

File: resources/robots/mini_cheetah/urdf/mini_cheetah_simple.urdf (robot description, URDF)
Before this commit: robot mini_cheetah, 22 links, 21 joints
Links:
- removed link fl_foot
- removed link fl_hip
- removed link fl_pastern
- removed link fl_shank
- removed link fl_thigh
- removed link fr_foot
- removed link fr_hip
- removed link fr_pastern
- removed link fr_shank
- removed link fr_thigh
- removed link hl_foot
- removed link hl_hip
- removed link hl_pastern
- removed link hl_shank
- removed link hl_thigh
- removed link hr_foot
- removed link hr_hip
- removed link hr_pastern
- removed link hr_shank
- removed link hr_thigh
- added link lf_foot, mass 0.20; collision cylinder length=0.02 radius=0.05; visual cylinder length=0.02 radius=0.05
- added link lf_hip, mass 4.558; visual cylinder length=0.05 radius=0.075
- added link lf_pastern, mass 0.875; collision cylinder length=0.15 radius=0.03; visual cylinder length=0.15 radius=0.03
- added link lf_shank, mass 1.404; collision cylinder length=0.25 radius=0.04; visual cylinder length=0.25 radius=0.04
- added link lf_thigh, mass 4.558; collision cylinder length=0.2 radius=0.075; visual cylinder length=0.2 radius=0.075
- added link lh_foot, mass 0.20; collision cylinder length=0.04 radius=0.05; visual cylinder length=0.04 radius=0.05
- added link lh_hip, mass 4.558; visual cylinder length=0.05 radius=0.075
- added link lh_pastern, mass 0.875; collision cylinder length=0.25 radius=0.03; visual cylinder length=0.25 radius=0.03
- added link lh_shank, mass 1.404; collision cylinder length=0.2 radius=0.04; visual cylinder length=0.2 radius=0.04
- added link lh_thigh, mass 4.558; collision cylinder length=0.2 radius=0.09; visual cylinder length=0.2 radius=0.09
- added link rf_foot, mass 0.20; collision cylinder length=0.02 radius=0.05; visual cylinder length=0.02 radius=0.05
- added link rf_hip, mass 4.558; visual cylinder length=0.05 radius=0.075
- added link rf_pastern, mass 0.875; collision cylinder length=0.15 radius=0.03; visual cylinder length=0.15 radius=0.03
- added link rf_shank, mass 1.404; collision cylinder length=0.25 radius=0.04; visual cylinder length=0.25 radius=0.04
- added link rf_thigh, mass 4.558; collision cylinder length=0.2 radius=0.075; visual cylinder length=0.2 radius=0.075
- added link rh_foot, mass 0.20; collision cylinder length=0.04 radius=0.05; visual cylinder length=0.04 radius=0.05
- added link rh_hip, mass 4.558; visual cylinder length=0.05 radius=0.075
- added link rh_pastern, mass 0.875; collision cylinder length=0.25 radius=0.03; visual cylinder length=0.25 radius=0.03
- added link rh_shank, mass 1.404; collision cylinder length=0.2 radius=0.04; visual cylinder length=0.2 radius=0.04
- added link rh_thigh, mass 4.558; collision cylinder length=0.2 radius=0.09; visual cylinder length=0.2 radius=0.09
Joints:
- removed joint 1_fr_haa
- removed joint 2_fl_haa
- removed joint 3_hr_haa
- removed joint 4_hl_haa
- removed joint base_joint
- removed joint fl_hfe
- removed joint fl_kfe
- removed joint fl_pastern_to_foot
- removed joint fl_pfe
- removed joint fr_hfe
- removed joint fr_kfe
- removed joint fr_pastern_to_foot
- removed joint fr_pfe
- removed joint hl_hfe
- removed joint hl_kfe
- removed joint hl_pastern_to_foot
- removed joint hl_pfe
- removed joint hr_hfe
- removed joint hr_kfe
- removed joint hr_pastern_to_foot
- removed joint hr_pfe
- added joint 0_base_joint: type revolute, parent front_base, child back_base, origin xyz=-0.5 0 0.3 rpy=0 0 0, axis 0 1 0, limit lower=-0.2 upper=0.2 effort=1100 velocity=41
- added joint 1_rh_haa: type revolute, parent back_base, child rh_hip, origin xyz=-0.3 -0.225 -0.4 rpy=0 3.141592 0, axis 1 0 0, limit lower=-0.2 upper=0.2 effort=1000 velocity=41
- added joint 2_lh_haa: type revolute, parent back_base, child lh_hip, origin xyz=-0.3 0.225 -0.4 rpy=0 3.141592 0, axis -1 0 0, limit lower=-0.2 upper=0.2 effort=1000 velocity=41
- added joint 3_rf_haa: type revolute, parent front_base, child rf_hip, origin xyz=0.35 -0.225 -0.23 rpy=0 0 0, axis -1 0 0, limit lower=-0.2 upper=0.2 effort=1000 velocity=41
- added joint 4_lf_haa: type revolute, parent front_base, child lf_hip, origin xyz=0.35 0.225 -0.23 rpy=0 0 0, axis 1 0 0, limit lower=-0.2 upper=0.2 effort=1000 velocity=41
- added joint lf_hfe: type revolute, parent lf_hip, child lf_thigh, origin xyz=0.0 0.12 -0.05 rpy=0.0 0.6 0.0, axis 0 1 0, limit lower=-0.7 upper=0.6 effort=700 velocity=41
- added joint lf_kfe: type revolute, parent lf_thigh, child lf_shank, origin xyz=0.0 0.0 -0.45 rpy=0.0 -0.6 0.0, axis 0 1 0, limit lower=-1.3 upper=0.1 effort=1000 velocity=26.8
- added joint lf_pastern_to_foot: type revolute, parent lf_pastern, child lf_foot, origin xyz=0.025 0.0 -0.3 rpy=0.0 0.0 0.0, axis 0 1 0, limit lower=-0.3 upper=1.8 effort=300 velocity=2.0
- added joint lf_pfe: type revolute, parent lf_shank, child lf_pastern, origin xyz=0.0 0.0 -0.3 rpy=0.05 0 0.0, axis 0 1 0, limit lower=-0.3 upper=2.2 effort=500 velocity=26.8
- added joint lh_hfe: type revolute, parent lh_hip, child lh_thigh, origin xyz=0.0 0.12 -0.05 rpy=0.0 2.841592 0.0, axis 0 1 0, limit lower=-0.7 upper=1.5 effort=700 velocity=41
- added joint lh_kfe: type revolute, parent lh_thigh, child lh_shank, origin xyz=0.0 0.0 -0.5 rpy=0.0 0.65 0.0, axis 0 1 0, limit lower=-0.2 upper=0.8 effort=1000 velocity=26.8
- added joint lh_pastern_to_foot: type revolute, parent lh_pastern, child lh_foot, origin xyz=0.0 0.0 -0.35 rpy=0.0 0.0 0.0, axis 0 1 0, limit lower=-0.3 upper=1.8 effort=300 velocity=2.0
- added joint lh_pfe: type revolute, parent lh_shank, child lh_pastern, origin xyz=-0.045 0.0 -0.35 rpy=0.0 -0.35 0.0, axis 0 1 0, limit lower=-0.3 upper=2.5 effort=500 velocity=26.8
- added joint rf_hfe: type revolute, parent rf_hip, child rf_thigh, origin xyz=0.0 -0.12 -0.05 rpy=0.0 0.6 0.0, axis 0 1 0, limit lower=-0.7 upper=0.6 effort=700 velocity=41
- added joint rf_kfe: type revolute, parent rf_thigh, child rf_shank, origin xyz=0.0 0.0 -0.45 rpy=0.0 -0.6 0.0, axis 0 1 0, limit lower=-1.3 upper=0.1 effort=1000 velocity=26.8
- added joint rf_pastern_to_foot: type revolute, parent rf_pastern, child rf_foot, origin xyz=0.025 0.0 -0.3 rpy=0.0 0.0 0.0, axis 0 1 0, limit lower=-0.3 upper=1.8 effort=300 velocity=2.0
- added joint rf_pfe: type revolute, parent rf_shank, child rf_pastern, origin xyz=0.0 0.0 -0.3 rpy=0.05 0 0.0, axis 0 1 0, limit lower=-0.3 upper=2.2 effort=500 velocity=26.8
- added joint rh_hfe: type revolute, parent rh_hip, child rh_thigh, origin xyz=0.0 -0.12 -0.05 rpy=0.0 2.841592 0.0, axis 0 1 0, limit lower=-0.7 upper=1.5 effort=700 velocity=41
- added joint rh_kfe: type revolute, parent rh_thigh, child rh_shank, origin xyz=0.0 0.0 -0.5 rpy=0.0 0.65 0.0, axis 0 1 0, limit lower=-0.2 upper=0.8 effort=1000 velocity=26.8
- added joint rh_pastern_to_foot: type revolute, parent rh_pastern, child rh_foot, origin xyz=0.0 0.0 -0.35 rpy=0.0 0.0 0.0, axis 0 1 0, limit lower=-0.3 upper=1.8 effort=300 velocity=2.0
- added joint rh_pfe: type revolute, parent rh_shank, child rh_pastern, origin xyz=-0.045 0.0 -0.35 rpy=0.0 -0.35 0.0, axis 0 1 0, limit lower=-0.3 upper=2.5 effort=500 velocity=26.8

Commit message: update scaling

File: resources/robots/mini_cheetah/urdf/mini_cheetah_simple.urdf (robot description, URDF)
Before this commit: robot mini_cheetah, 22 links, 21 joints
Joints:
- joint lf_hfe: limit lower=-0.7 upper=0.6 effort=700 velocity=41 -> lower=-0.7 upper=0.6 effort=1000 velocity=41
- joint lh_hfe: limit lower=-0.7 upper=1.5 effort=700 velocity=41 -> lower=-0.7 upper=1.5 effort=1000 velocity=41
- joint rf_hfe: limit lower=-0.7 upper=0.6 effort=700 velocity=41 -> lower=-0.7 upper=0.6 effort=1000 velocity=41
- joint rh_hfe: limit lower=-0.7 upper=1.5 effort=700 velocity=41 -> lower=-0.7 upper=1.5 effort=1000 velocity=41
