Commit message: split off horse on its own

File: resources/robots/mini_cheetah/urdf/mini_cheetah_simple.urdf (robot description, URDF)
Before this commit: robot mini_cheetah, 22 links, 21 joints
Links:
- removed link back_base
- removed link front_base
- removed link lf_pastern
- removed link lh_pastern
- removed link rf_pastern
- removed link rh_pastern
- added link base, mass 3.3; collision box size=0.30 0.20 0.10; visual mesh filename=meshes/mini_vision_body.dae
- link lf_foot: mass 0.20 -> 0.01; geometry collision sphere radius=0.0202
- link lf_hip: mass 4.558 -> 0.54; geometry visual mesh filename=meshes/mini_vision_abd.dae
- link lf_shank: mass 1.404 -> 0.064; geometry collision cylinder length=0.1 radius=0.01; visual mesh filename=meshes/lower_leg.dae
- link lf_thigh: mass 4.558 -> 0.634; geometry collision cylinder length=0.17 radius=0.015; visual mesh filename=meshes/mini_vision_upper_leg.dae
- link lh_foot: mass 0.20 -> 0.01; geometry collision sphere radius=0.0202
- link lh_hip: mass 4.558 -> 0.54; geometry visual mesh filename=meshes/mini_vision_abd.dae
- link lh_shank: mass 1.404 -> 0.064; geometry collision cylinder length=0.1 radius=0.01; visual mesh filename=meshes/lower_leg.dae
- link lh_thigh: mass 4.558 -> 0.634; geometry collision cylinder length=0.17 radius=0.015; visual mesh filename=meshes/mini_vision_upper_leg.dae
- link rf_foot: mass 0.20 -> 0.01; geometry collision sphere radius=0.0202
- link rf_hip: mass 4.558 -> 0.54; geometry visual mesh filename=meshes/mini_vision_abd.dae
- link rf_shank: mass 1.404 -> 0.064; geometry collision cylinder length=0.1 radius=0.01; visual mesh filename=meshes/lower_leg.dae
- link rf_thigh: mass 4.558 -> 0.634; geometry collision cylinder length=0.17 radius=0.015; visual mesh filename=meshes/mini_vision_upper_leg.dae
- link rh_foot: mass 0.20 -> 0.01; geometry collision sphere radius=0.0202
- link rh_hip: mass 4.558 -> 0.54; geometry visual mesh filename=meshes/mini_vision_abd.dae
- link rh_shank: mass 1.404 -> 0.064; geometry collision cylinder length=0.1 radius=0.01; visual mesh filename=meshes/lower_leg.dae
- link rh_thigh: mass 4.558 -> 0.634; geometry collision cylinder length=0.17 radius=0.015; visual mesh filename=meshes/mini_vision_upper_leg.dae
Joints:
- removed joint 0_base_joint
- removed joint 1_rh_haa
- removed joint 2_lh_haa
- removed joint 3_rf_haa
- removed joint 4_lf_haa
- removed joint lf_pastern_to_foot
- removed joint lf_pfe
- removed joint lh_pastern_to_foot
- removed joint lh_pfe
- removed joint rf_pastern_to_foot
- removed joint rf_pfe
- removed joint rh_pastern_to_foot
- removed joint rh_pfe
- added joint 1_rf_haa: type revolute, parent base, child rf_hip, origin xyz=0.14775 -0.049 0.0 rpy=0 0 0, axis 1 0 0, limit lower=-1.5 upper=1.5 effort=18 velocity=41
- added joint 2_lf_haa: type revolute, parent base, child lf_hip, origin xyz=0.14775 0.049 0.0 rpy=0 0 0, axis 1 0 0, limit lower=-1.5 upper=1.5 effort=18 velocity=41
- added joint 3_rh_haa: type revolute, parent base, child rh_hip, origin xyz=-0.14775 -0.049 0.0 rpy=0 3.141592 0, axis -1 0 0, limit lower=-1.5 upper=1.5 effort=18 velocity=41
- added joint 4_lh_haa: type revolute, parent base, child lh_hip, origin xyz=-0.14775 0.049 0.0 rpy=0 3.141592 0, axis -1 0 0, limit lower=-1.5 upper=1.5 effort=18 velocity=41
- added joint lf_shank_to_foot: type fixed, parent lf_shank, child lf_foot, origin xyz=0.0 0.0 -0.22 rpy=0.0 0.0 0.0
- added joint lh_shank_to_foot: type fixed, parent lh_shank, child lh_foot, origin xyz=0.0 0.0 -0.22 rpy=0.0 0.0 0.0
- added joint rf_shank_to_foot: type fixed, parent rf_shank, child rf_foot, origin xyz=0.0 0.0 -0.22 rpy=0.0 0.0 0.0
- added joint rh_shank_to_foot: type fixed, parent rh_shank, child rh_foot, origin xyz=0.0 0.0 -0.22 rpy=0.0 0.0 0.0
- joint lf_hfe: axis 0 1 0 -> 0 -1 0; limit lower=-0.7 upper=0.6 effort=1000 velocity=41 -> lower=-2.6 upper=2.6 effort=18 velocity=41; origin xyz=0.0 0.12 -0.05 rpy=0.0 0.6 0.0 -> xyz=0.055 0.019 0.00 rpy=0.0 0.0 0.0
- joint lf_kfe: axis 0 1 0 -> 0 -1 0; limit lower=-1.3 upper=0.1 effort=1000 velocity=26.8 -> lower=-2.7 upper=2.7 effort=28 velocity=26.8; origin xyz=0.0 0.0 -0.45 rpy=0.0 -0.6 0.0 -> xyz=0.0 0.049 -0.2085 rpy=0.0 0 0.0
- joint lh_hfe: axis 0 1 0 -> 0 -1 0; limit lower=-0.7 upper=1.5 effort=1000 velocity=41 -> lower=-2.6 upper=2.6 effort=18 velocity=41; origin xyz=0.0 0.12 -0.05 rpy=0.0 2.841592 0.0 -> xyz=0.055 0.019 0.00 rpy=0.0 3.141592 0.0
- joint lh_kfe: axis 0 1 0 -> 0 -1 0; limit lower=-0.2 upper=0.8 effort=1000 velocity=26.8 -> lower=-2.7 upper=2.7 effort=28 velocity=26.8; origin xyz=0.0 0.0 -0.5 rpy=0.0 0.65 0.0 -> xyz=0.0 0.049 -0.2085 rpy=0.0 0 0.0
- joint rf_hfe: axis 0 1 0 -> 0 -1 0; limit lower=-0.7 upper=0.6 effort=1000 velocity=41 -> lower=-2.6 upper=2.6 effort=18 velocity=41; origin xyz=0.0 -0.12 -0.05 rpy=0.0 0.6 0.0 -> xyz=0.055 -0.019 0.00 rpy=0.0 0.0 0.0
- joint rf_kfe: axis 0 1 0 -> 0 -1 0; limit lower=-1.3 upper=0.1 effort=1000 velocity=26.8 -> lower=-2.7 upper=2.7 effort=28 velocity=26.8; origin xyz=0.0 0.0 -0.45 rpy=0.0 -0.6 0.0 -> xyz=0.0 -0.049 -0.2085 rpy=0.0 0 0.0
- joint rh_hfe: axis 0 1 0 -> 0 -1 0; limit lower=-0.7 upper=1.5 effort=1000 velocity=41 -> lower=-2.6 upper=2.6 effort=18 velocity=41; origin xyz=0.0 -0.12 -0.05 rpy=0.0 2.841592 0.0 -> xyz=0.055 -0.019 0.00 rpy=0.0 3.141592 0.0
- joint rh_kfe: axis 0 1 0 -> 0 -1 0; limit lower=-0.2 upper=0.8 effort=1000 velocity=26.8 -> lower=-2.7 upper=2.7 effort=28 velocity=26.8; origin xyz=0.0 0.0 -0.5 rpy=0.0 0.65 0.0 -> xyz=0.0 -0.049 -0.2085 rpy=0.0 0 0.0
