Commit message: some tuning, mainly for back stiffness/torque limits, and weights. Also increased sim frequency for smoother joint tracking

File: resources/robots/horse/urdf/horse.urdf (robot description, URDF)
Before this commit: robot mini_cheetah, 22 links, 21 joints
Joints:
- joint 0_base_joint: limit lower=-0.2 upper=0.2 effort=1100 velocity=41 -> lower=-0.2 upper=0.2 effort=10000 velocity=41

Commit message: expand joint limits for lay down motion

File: resources/robots/horse/urdf/horse.urdf (robot description, URDF)
Before this commit: robot mini_cheetah, 22 links, 21 joints
Joints:
- joint 1_rh_haa: origin xyz=-0.3 -0.225 -0.4 rpy=0 3.141592 0 -> xyz=-0.3 -0.225 -0.15 rpy=0 3.141592 0
- joint 2_lh_haa: origin xyz=-0.3 0.225 -0.4 rpy=0 3.141592 0 -> xyz=-0.3 0.225 -0.15 rpy=0 3.141592 0
- joint 3_rf_haa: origin xyz=0.35 -0.225 -0.23 rpy=0 0 0 -> xyz=0.35 -0.225 0.0 rpy=0 0 0
- joint 4_lf_haa: origin xyz=0.35 0.225 -0.23 rpy=0 0 0 -> xyz=0.35 0.225 0.0 rpy=0 0 0
- joint lf_hfe: limit lower=-0.7 upper=0.6 effort=1000 velocity=41 -> lower=-1.0 upper=0.6 effort=1000 velocity=41
- joint lf_kfe: limit lower=-1.3 upper=0.1 effort=1000 velocity=26.8 -> lower=-1.5 upper=0.1 effort=1000 velocity=26.8
- joint lf_pfe: limit lower=-0.3 upper=2.2 effort=500 velocity=26.8 -> lower=-0.3 upper=3.0 effort=500 velocity=26.8
- joint lh_hfe: limit lower=-0.7 upper=1.5 effort=1000 velocity=41 -> lower=-1.5 upper=0.5 effort=1000 velocity=41
- joint lh_kfe: limit lower=-0.2 upper=0.8 effort=1000 velocity=26.8 -> lower=-0.2 upper=1.0 effort=1000 velocity=26.8
- joint lh_pfe: limit lower=-0.3 upper=2.5 effort=500 velocity=26.8 -> lower=-1.2 upper=2.5 effort=500 velocity=26.8
- joint rf_hfe: limit lower=-0.7 upper=0.6 effort=1000 velocity=41 -> lower=-1.0 upper=0.6 effort=1000 velocity=41
- joint rf_kfe: limit lower=-1.3 upper=0.1 effort=1000 velocity=26.8 -> lower=-1.5 upper=0.1 effort=1000 velocity=26.8
- joint rf_pfe: limit lower=-0.3 upper=2.2 effort=500 velocity=26.8 -> lower=-0.3 upper=3.0 effort=500 velocity=26.8
- joint rh_hfe: limit lower=-0.7 upper=1.5 effort=1000 velocity=41 -> lower=-1.5 upper=0.5 effort=1000 velocity=41
- joint rh_kfe: limit lower=-0.2 upper=0.8 effort=1000 velocity=26.8 -> lower=-0.2 upper=1.0 effort=1000 velocity=26.8
- joint rh_pfe: limit lower=-0.3 upper=2.5 effort=500 velocity=26.8 -> lower=-1.2 upper=2.5 effort=500 velocity=26.8

Commit message: plots and fix height pos and command

File: resources/robots/horse/urdf/horse.urdf (robot description, URDF)
Before this commit: robot mini_cheetah, 22 links, 21 joints
Links:
- added link top, mass 1; collision box size=1.45 0.4 0.1; visual box size=1.45 0.4 0.1
- link front_base: geometry collision box size=.8 0.3 0.51; visual box size=0.8 0.38 0.61
Joints:
- added joint dummy_joint: type fixed, parent top, child front_base, origin xyz=0 0 0 rpy=0 0 0, axis 0 0 0, limit lower=0 upper=0 effort=0 velocity=0

Commit message: Revert "plots and fix height pos and command"
This reverts commit 1957e3f5fdcd221bfc547ace0ca1f2b524d6d337.

File: resources/robots/horse/urdf/horse.urdf (robot description, URDF)
Before this commit: robot mini_cheetah, 23 links, 22 joints
Links:
- removed link top
- link front_base: geometry collision box size=.8 0.38 0.51; visual box size=0.8 0.38 0.61
Joints:
- removed joint dummy_joint

Commit message: best result: switch_height

File: resources/robots/horse/urdf/horse.urdf (robot description, URDF)
Before this commit: robot mini_cheetah, 22 links, 21 joints
Links:
- added link top, mass 1; collision box size=1.45 0.4 0.1; visual box size=1.45 0.4 0.1
Joints:
- added joint dummy_joint: type fixed, parent top, child front_base, origin xyz=0 0 0 rpy=0 0 0, axis 0 0 0, limit lower=0 upper=0 effort=0 velocity=0
