Commit message: Tweaks (#247)
* bug fixes (#239)

* precommit check against large files and merge conflict code (#240)

* format ETA in the logger to hours:minutes:seconds (#242)

* lots of tweaks, trains well now for both

* merge lqc_j

---------

Co-authored-by: Julianna Schneider <54411881+jschneider03@users.noreply.github.com>

File: resources/robots/pendulum/urdf/pendulum.urdf (robot description, URDF)
Before this commit: robot pendulum, 2 links, 1 joints
Links:
- link pole: mass 2 -> 1
Joints:
- joint theta: limit effort=0.5 -> effort=5.0

Commit message: match URDF, obs, ctrl freq, etc to gymansium

File: resources/robots/pendulum/urdf/pendulum.urdf (robot description, URDF)
Before this commit: robot pendulum, 2 links, 1 joints
Joints:
- joint theta: limit effort=5.0 -> effort=2.0

Commit message: WIP: fix polyak bug, some more tuning

File: resources/robots/pendulum/urdf/pendulum.urdf (robot description, URDF)
Before this commit: robot pendulum, 2 links, 1 joints
Joints:
- joint theta: limit effort=2.0 -> effort=5.0

Commit message: WIP: works on CPU, not GPU (nvidia warp)

File: resources/robots/pendulum/urdf/pendulum.urdf (robot description, URDF)
Before this commit: robot pendulum, 2 links, 1 joints
Joints:
- joint theta: limit effort=5.0 -> effort=5.0 velocity=100.0
